File: oshe_dmm_KiCAD/oshe_dmm_project_v1/oshe_dmm_project_v1.kicad_sch (KiCad schematic)
At the start: 1 part, among them U1 ATmega328P-A

Commit message: Added BMS to schematic
Parts:
- added BAT+1, BAT-1, Thermistor1: Pad, TestPoint:TestPoint_Pad_4.0x4.0mm, symbol Connector:TestPoint
- added C1, C2: 22pF, Capacitor_SMD:C_1206_3216Metric_Pad1.33x1.80mm_HandSolder, symbol Device:C
- added C3, C4, C6: 10uF, symbol Device:C
- added C5: 0.1uF, symbol Device:C_Polarized_US
- added C7: C, symbol Device:C
- added C8: 1.0uF, symbol Device:C_Polarized_US
- added D1, D3: 1N4002, Diode_THT:D_DO-41_SOD81_P10.16mm_Horizontal, symbol Diode:1N4002
- added D2: PGOOD, LED_SMD:LED_1206_3216Metric_Pad1.42x1.75mm_HandSolder, symbol Device:LED
- added D4: CHG, LED_SMD:LED_1206_3216Metric_Pad1.42x1.75mm_HandSolder, symbol Device:LED
- added J1: USB_C_Receptacle_USB2.0_14P, symbol Connector:USB_C_Receptacle_USB2.0_14P
- added JP1, JP2: SolderJumper_3_Open, Jumper:SolderJumper-3_P1.3mm_Open_Pad1.0x1.5mm, symbol Jumper:SolderJumper_3_Open
- added JP3: SolderJumper_3_Open, symbol Jumper:SolderJumper_2_Open
- added R1: 10k, symbol Device:R_US
- added R2: 1.24k, symbol Device:R_US
- added R3: 49.9k, symbol Device:R_US
- added R4: 1.07k, symbol Device:R_US
- added R5: 750, symbol Device:R_US
- added R6: ?, symbol Device:R_US
- added R7: 240, symbol Device:R_US
- added R8, R9: 1.5k, Resistor_SMD:R_1206_3216Metric_Pad1.30x1.75mm_HandSolder, symbol Device:R_US
- added SW1: SW_Push, symbol Switch:SW_Push
- added SW2: SW_SPST, symbol Switch:SW_SPST
- added U2: BQ24075RGT, Package_DFN_QFN:VQFN-16-1EP_3x3mm_P0.5mm_EP1.6x1.6mm, symbol Battery_Management:BQ24075RGT
- added U3: LM317_SOT-223, Package_TO_SOT_SMD:SOT-223-3_TabPin2, symbol Regulator_Linear:LM317_SOT-223
- added Y1: 16MHz, symbol Device:Crystal
Connections:
- net +5V: now reaches U1.18 (AVCC)
- net +5V: now also U1.4 (VCC), U1.6 (VCC), C8.1, D1.2 (A), D3.1 (K), JP2.1 (A), JP3.2 (B), R1.2, R7.1, U3.2 (VO)
- net GND: now reaches U1.21 (GND), U1.3 (GND), U1.5 (GND)
- net GND: now also BAT-1.1, C1.2, C2.1, C3.2, C4.2, C5.2, C6.2, C7.2, C8.2, J1.A1 (GND), J1.A12 (GND), J1.B1 (GND), J1.B12 (GND), R1.1, R2.2, R3.2, R4.2, R5.2, R6.2, SW1.2, U2.17 (VSS), U2.4 (~{CE}), U2.6 (EN1), U2.8 (VSS)
- net SDA: now reaches U1.27 (PC4)
- net SCL: now reaches U1.28 (PC5)
- net at U1.29 (~{RESET}/PC6): now also SW1.1
- net RXD: now reaches U1.30 (PD0)
- net TXD: now reaches U1.31 (PD1)
- net at U1.7 (XTAL1/PB6): now also C1.1, Y1.2
- net at U1.8 (XTAL2/PB7): now also C2.2, Y1.1
- new net: BAT+1.1, C3.1, JP1.2 (C)
- new net: D4.2 (A), R9.2
- new net: C5.1, D1.1 (K), JP2.3 (B), U3.3 (VI)
- new net: C7.1, D3.2 (A), R6.1, R7.2, U3.1 (ADJ)
- new net: JP2.2 (C), SW2.2 (B)
- new net: D4.1 (K), U2.9 (~{CHG})
- new net: D2.1 (K), U2.7 (~{PGOOD})
- new net: D2.2 (A), R8.2
- new net 9V_BAT_IN: C6.1, JP1.3 (B), R8.1, R9.1, SW2.1 (A), U2.10 (OUT), U2.11 (OUT)
- new net BMS_BAT_IN: JP1.1 (A), U2.2 (BAT), U2.3 (BAT)
- new net R-ILIM: R4.1, U2.12 (ILIM)
- new net R-ISET: R5.1, U2.16 (ISET)
- new net R-ITERM: R2.1, U2.15 (SYSOFF)
- new net R-TMR: R3.1, U2.14 (TMR)
- new net TS: Thermistor1.1, U2.1 (TS)
- new net USB_Power_IN: C4.1, J1.A4 (VBUS), J1.A9 (VBUS), J1.B4 (VBUS), J1.B9 (VBUS), JP3.1 (A), U2.13 (IN), U2.5 (EN2)
Other:
- note added: "ATMEGA328P-AU Microcontroller"
- note added: "NOTES:"
- note added: "Original circuit built on the BQ24074RGTR from Texas Instruments Configured for 1.2A Fast Charge"
- moved on the sheet: U1

Commit message: Updated main schematic
Parts:
- added C1, C2, C5: 0.1uF, Capacitor_SMD:C_1206_3216Metric_Pad1.33x1.80mm_HandSolder, symbol Device:C
- added D1: Green, LED_SMD:LED_1206_3216Metric_Pad1.42x1.75mm_HandSolder, symbol Device:LED
- added J1: FTDI Basic, Connector_PinSocket_2.54mm:PinSocket_1x06_P2.54mm_Vertical, symbol Connector_Generic:Conn_01x06
- added R1: 330, symbol Device:R_US
- renumbered C7 to C10, C8 to C11, C1 to C3, C2 to C4, C3 to C6, C4 to C7, C5 to C8, C6 to C9, D1 to D3, D3 to D5, J1 to J2, R9 to R10, R1 to R2, R2 to R3, R3 to R4, R4 to R5, R5 to R6, R6 to R7, R7 to R9
Connections:
- net +5V: now also C2.1, J1.4 (Pin_4)
- net GND: now also SW1.1, C1.1, C2.2, D1.1 (K), J1.5 (Pin_5), J1.6 (Pin_6); no longer R2.1, SW1.2
- net RXD: now also J1.3 (Pin_3)
- net TXD: now also J1.2 (Pin_2)
- net D3: now reaches U1.1 (PD3)
- net D6: now reaches U1.10 (PD6)
- net D7: now reaches U1.11 (PD7)
- net D8: now reaches U1.12 (PB0)
- net D9: now reaches U1.13 (PB1)
- net D10: now reaches U1.14 (PB2)
- net MOSI/D11: now reaches U1.15 (PB3)
- net MISO/D12: now reaches U1.16 (PB4)
- net SCK/D13: now reaches U1.17 (PB5)
- net SCK/D13: now also R1.2
- net A6: now reaches U1.19 (ADC6)
- net D4: now reaches U1.2 (PD4)
- net at U1.20 (AREF): now also C1.2
- net A7: now reaches U1.22 (ADC7)
- net A0: now reaches U1.23 (PC0)
- net A1: now reaches U1.24 (PC1)
- net A2: now reaches U1.25 (PC2)
- net A3: now reaches U1.26 (PC3)
- net at U1.29 (~{RESET}/PC6): now also R2.1, SW1.2, C5.1; no longer SW1.1
- net D2: now reaches U1.32 (PD2)
- net D5: now reaches U1.9 (PD5)
- new net: D1.2 (A), R1.1
- new net DTR: C5.2, J1.1 (Pin_1)
Other:
- note added: "Battery Management System"
- note removed: "NOTES:"
- note removed: "Original circuit built on the BQ24074RGTR from Texas Instruments Configured for 1.2A Fast Charge"
- moved on the sheet: BAT+1, BAT-1, C10, C11, C3, C4, C6, C7, C8, C9, D2, D3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

Commit message: Created an initial PCB
Parts:
- C10, C11, C6, C7, C8, C9: footprint (none) -> Capacitor_SMD:C_1206_3216Metric_Pad1.33x1.80mm_HandSolder
- J2: footprint (none) -> Connector_USB:USB_C_Receptacle_Molex_105450-0101
- JP1, JP2: footprint Jumper:SolderJumper-3_P1.3mm_Open_Pad1.0x1.5mm -> Jumper:SolderJumper-3_P1.3mm_Open_Pad1.0x1.5mm_NumberLabels
- JP3: value SolderJumper_3_Open -> SolderJumper_2_Open; footprint (none) -> Jumper:SolderJumper-2_P1.3mm_Open_Pad1.0x1.5mm
- R1, R2, R3, R4, R5, R6, R7, R9: footprint (none) -> Resistor_SMD:R_1206_3216Metric_Pad1.30x1.75mm_HandSolder
- SW1: footprint (none) -> Button_Switch_SMD:SW_Push_1P1T-MP_NO_Horizontal_Alps_SKRTLAE010
- SW2: footprint (none) -> Button_Switch_SMD:SW_SPST_B3S-1000
- Y1: footprint (none) -> Crystal:Resonator_Murata_CSTLSxxxG-3Pin_W8.0mm_H3.0mm
Changed lines of the file:
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@@
 			)
 		)
-		(property "Footprint" "Jumper:SolderJumper-3_P1.3mm_Open_Pad1.0x1.5mm"
+		(property "Footprint" "Jumper:SolderJumper-3_P1.3mm_Open_Pad1.0x1.5mm_NumberLabels"
 			(at 373.38 105.41 0)
 			(effects
@@
 			)
 		)
-		(property "Footprint" ""
+		(property "Footprint" "Resistor_SMD:R_1206_3216Metric_Pad1.30x1.75mm_HandSolder"
 			(at 431.546 81.534 90)
 			(effects
@@
 			)
 		)
-		(property "Footprint" ""
+		(property "Footprint" "Resistor_SMD:R_1206_3216Metric_Pad1.30x1.75mm_HandSolder"
 			(at 411.226 81.534 90)
 			(effects
@@
 			)
 		)
-		(property "Footprint" ""
+		(property "Footprint" "Capacitor_SMD:C_1206_3216Metric_Pad1.33x1.80mm_HandSolder"
 			(at 514.0452 49.53 0)
 			(effects
@@
 			)
 		)
-		(property "Footprint" ""
+		(property "Footprint" "Capacitor_SMD:C_1206_3216Metric_Pad1.33x1.80mm_HandSolder"
 			(at 358.4448 114.3 0)
 			(effects
@@
 			)
 		)
-		(property "Value" "SolderJumper_3_Open"
+		(property "Value" "SolderJumper_2_Open"
 			(at 551.18 90.1699 90)
 			(effects
@@
 			)
 		)
-		(property "Footprint" ""
+		(property "Footprint" "Jumper:SolderJumper-2_P1.3mm_Open_Pad1.0x1.5mm"
 			(at 548.64 88.9 0)
 			(effects
@@
 			)
 		)
-		(property "Footprint" ""
+		(property "Footprint" "Capacitor_SMD:C_1206_3216Metric_Pad1.33x1.80mm_HandSolder"
 			(at 509.27 111.76 0)
 			(effects
@@
 			)
 		)
-		(property "Footprint" ""
+		(property "Footprint" "Resistor_SMD:R_1206_3216Metric_Pad1.30x1.75mm_HandSolder"
 			(at 462.026 81.534 90)
 			(effects
@@
 			)
 		)
-		(property "Footprint" ""
+		(property "Footprint" "Button_Switch_SMD:SW_SPST_B3S-1000"
 			(at 455.93 110.49 0)
 			(effects
@@
 			)
 		)
-		(property "Footprint" ""
+		(property "Footprint" "Connector_USB:USB_C_Receptacle_Molex_105450-0101"
 			(at 351.79 48.26 0)
 			(effects
@@
 			)
 		)
-		(property "Footprint" ""
+		(property "Footprint" "Capacitor_SMD:C_1206_3216Metric_Pad1.33x1.80mm_HandSolder"
 			(at 543.2552 123.19 0)
 			(effects
@@
 			)
 		)
-		(property "Footprint" ""
+		(property "Footprint" "Capacitor_SMD:C_1206_3216Metric_Pad1.33x1.80mm_HandSolder"
 			(at 553.72 119.38 0)
 			(effects
@@
 			)
 		)
-		(property "Footprint" ""
+		(property "Footprint" "Capacitor_SMD:C_1206_3216Metric_Pad1.33x1.80mm_HandSolder"
 			(at 385.7752 45.72 0)
 			(effects
@@
 			)
 		)
-		(property "Footprint" ""
+		(property "Footprint" "Resistor_SMD:R_1206_3216Metric_Pad1.30x1.75mm_HandSolder"
 			(at 116.586 86.614 90)
 			(effects
@@
 			)
 		)
-		(property "Footprint" ""
+		(property "Footprint" "Button_Switch_SMD:SW_Push_1P1T-MP_NO_Horizontal_Alps_SKRTLAE010"
 			(at 85.09 86.36 0)
 			(effects
@@
 			)
 		)
-		(property "Footprint" "Jumper:SolderJumper-3_P1.3mm_Open_Pad1.0x1.5mm"
+		(property "Footprint" "Jumper:SolderJumper-3_P1.3mm_Open_Pad1.0x1.5mm_NumberLabels"
 			(at 476.25 110.49 0)
 			(effects
@@
 			)
 		)
-		(property "Footprint" ""
+		(property "Footprint" "Resistor_SMD:R_1206_3216Metric_Pad1.30x1.75mm_HandSolder"
 			(at 533.146 106.934 90)
 			(effects
@@
 			)
 		)
-		(property "Footprint" ""
+		(property "Footprint" "Resistor_SMD:R_1206_3216Metric_Pad1.30x1.75mm_HandSolder"
 			(at 522.986 119.634 90)
 			(effects
@@
 			)
 		)
-		(property "Footprint" ""
+		(property "Footprint" "Crystal:Resonator_Murata_CSTLSxxxG-3Pin_W8.0mm_H3.0mm"
 			(at 100.33 60.96 0)
 			(effects
@@
 			)
 		)
-		(property "Footprint" ""
+		(property "Footprint" "Resistor_SMD:R_1206_3216Metric_Pad1.30x1.75mm_HandSolder"
 			(at 102.616 38.354 90)
 			(effects
@@
 			)
 		)
-		(property "Footprint" ""
+		(property "Footprint" "Resistor_SMD:R_1206_3216Metric_Pad1.30x1.75mm_HandSolder"
 			(at 451.866 81.534 90)
 			(effects

Commit message: Made some changes to the PCB
Parts:
- SW2: value SW_SPST -> Power_Switch; footprint Button_Switch_SMD:SW_SPST_B3S-1000 -> Button_Switch_SMD:SW_SPDT_CK_JS102011SAQN
- renumbered C9 to C8, C8 to C9
Changed lines of the file:
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@@
 	)
 	(junction
+		(at 445.77 110.49)
+		(diameter 0)
+		(color 0 0 0 0)
+	)
+	(junction
 		(at 509.27 100.33)
 		(diameter 0)
@@
 	)
 	(junction
-		(at 445.77 110.49)
-		(diameter 0)
-		(color 0 0 0 0)
-	)
-	(junction
 		(at 548.64 100.33)
 		(diameter 0)
@@
 	(wire
 		(pts
+			(xy 440.69 105.41) (xy 445.77 105.41)
+		)
+		(stroke
+			(width 0)
+			(type default)
+		)
+	)
+	(wire
+		(pts
 			(xy 373.38 97.79) (xy 375.92 97.79)
 		)
@@
 	(wire
 		(pts
-			(xy 440.69 105.41) (xy 445.77 105.41)
+			(xy 440.69 110.49) (xy 445.77 110.49)
 		)
 		(stroke
@@
 	(wire
 		(pts
-			(xy 440.69 110.49) (xy 445.77 110.49)
-		)
-		(stroke
-			(width 0)
-			(type default)
-		)
-	)
-	(wire
-		(pts
 			(xy 410.21 88.9) (xy 410.21 91.44)
 		)
@@
 	)
 	(global_label "USB_Power_IN"
-		(shape input)
+		(shape output)
 		(at 397.51 29.21 0)
 		(fields_autoplaced yes)
@@
 	)
 	(global_label "BMS_Power_Out"
-		(shape input)
+		(shape output)
 		(at 547.37 38.1 0)
 		(fields_autoplaced yes)
@@
 	)
 	(global_label "9V_BAT_IN"
-		(shape input)
+		(shape output)
 		(at 375.92 113.03 0)
 		(fields_autoplaced yes)
@@
 	(global_label "9V_BAT_IN"
 		(shape input)
-		(at 440.69 110.49 180)
+		(at 440.69 105.41 180)
 		(fields_autoplaced yes)
 		(effects
@@
 		)
 		(property "Intersheetrefs" "${INTERSHEET_REFS}"
-			(at 428.21 110.49 0)
+			(at 428.21 105.41 0)
 			(effects
 				(font
@@
 	)
 	(global_label "BMS_BAT_IN"
-		(shape input)
+		(shape output)
 		(at 375.92 97.79 0)
 		(fields_autoplaced yes)
@@
 	(global_label "BMS_Power_Out"
 		(shape input)
-		(at 440.69 105.41 180)
+		(at 440.69 110.49 180)
 		(fields_autoplaced yes)
 		(effects
@@
 		)
 		(property "Intersheetrefs" "${INTERSHEET_REFS}"
-			(at 423.0092 105.41 0)
+			(at 423.0092 110.49 0)
 			(effects
 				(font
@@
 	)
 	(global_label "+5V"
-		(shape input)
+		(shape output)
 		(at 560.07 100.33 0)
 		(fields_autoplaced yes)
@@
 	)
 	(global_label "+5V"
-		(shape input)
+		(shape output)
 		(at 481.33 120.65 0)
 		(fields_autoplaced yes)
@@
 	)
 	(global_label "TS"
-		(shape input)
+		(shape output)
 		(at 359.41 95.25 0)
 		(fields_autoplaced yes)
@@
 		(dnp no)
 		(fields_autoplaced yes)
-		(property "Reference" "C9"
+		(property "Reference" "C8"
 			(at 516.89 44.4499 0)
 			(effects
@@
 			(project "oshe_dmm_project_v1"
 				(path "/24c8480a-c336-4df0-8536-7016ee8fc0ac"
-					(reference "C9")
+					(reference "C8")
 					(unit 1)
 				)
@@
 		(on_board yes)
 		(dnp no)
-		(property "Reference" "C8"
+		(property "Reference" "C9"
 			(at 513.08 109.8549 0)
 			(effects
@@
 			(project "oshe_dmm_project_v1"
 				(path "/24c8480a-c336-4df0-8536-7016ee8fc0ac"
-					(reference "C8")
+					(reference "C9")
 					(unit 1)
 				)
@@
 			)
 		)
-		(property "Value" "SW_SPST"
+		(property "Value" "Power_Switch"
 			(at 455.93 106.68 0)
 			(effects
@@
 			)
 		)
-		(property "Footprint" "Button_Switch_SMD:SW_SPST_B3S-1000"
+		(property "Footprint" "Button_Switch_SMD:SW_SPDT_CK_JS102011SAQN"
 			(at 455.93 110.49 0)
 			(effects

Commit message: Made more PCB changes
Parts:
- removed D3: 1N4002, Diode_THT:D_DO-41_SOD81_P10.16mm_Horizontal, symbol Diode:1N4002
- BAT+1, BAT-1, Thermistor1: footprint TestPoint:TestPoint_Pad_4.0x4.0mm -> TestPoint:TestPoint_THTPad_D4.0mm_Drill2.0mm
- C10: value C -> 10uF
- D4: renamed from D5; footprint Diode_THT:D_DO-41_SOD81_P10.16mm_Horizontal -> Diode_SMD:D_1206_3216Metric_Pad1.42x1.75mm_HandSolder
- R7: value ? -> 1.2k
- R9: value 240 -> 390
- renumbered C5 to C3, C3 to C4, C4 to C5, C9 to C8, C8 to C9, D4 to D3
Other:
- moved on the sheet: JP3

Commit message: Made more changes
Parts:
- removed R3: 1.24k, Resistor_SMD:R_1206_3216Metric_Pad1.30x1.75mm_HandSolder, symbol Device:R_US
- J2: footprint Connector_USB:USB_C_Receptacle_Molex_105450-0101 -> Connector_USB:USB_C_Receptacle_GCT_USB4085
- renumbered R4 to R3, R5 to R4, R6 to R5, R7 to R6, R8 to R7, R9 to R8, R10 to R9
Connections:
- net R-ITERM is gone; now on net GND: U2.15 (SYSOFF)
Changed lines of the file:
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@@
 	(wire
 		(pts
-			(xy 410.21 88.9) (xy 410.21 85.09)
-		)
-		(stroke
-			(width 0)
-			(type default)
-		)
-	)
-	(wire
-		(pts
 			(xy 472.44 110.49) (xy 461.01 110.49)
 		)
@@
 	(wire
 		(pts
-			(xy 410.21 45.72) (xy 410.21 77.47)
+			(xy 410.21 45.72) (xy 410.21 88.9)
 		)
 		(stroke
@@
 		)
 	)
-	(label "R-ITERM"
-		(at 410.21 77.47 0)
-		(fields_autoplaced yes)
-		(effects
-			(font
-				(size 1.27 1.27)
-			)
-			(justify left bottom)
-		)
-	)
 	(label "R-ISET"
 		(at 461.01 77.47 0)
@@
 		(dnp no)
 		(fields_autoplaced yes)
-		(property "Reference" "R4"
+		(property "Reference" "R3"
 			(at 433.07 80.0099 0)
 			(effects
@@
 			(project "oshe_dmm_project_v1"
 				(path "/24c8480a-c336-4df0-8536-7016ee8fc0ac"
-					(reference "R4")
+					(reference "R3")
 					(unit 1)
 				)
@@
 		(dnp no)
 		(fields_autoplaced yes)
-		(property "Reference" "R10"
+		(property "Reference" "R9"
 			(at 539.75 44.4499 0)
 			(effects
@@
 			(project "oshe_dmm_project_v1"
 				(path "/24c8480a-c336-4df0-8536-7016ee8fc0ac"
-					(reference "R10")
+					(reference "R9")
 					(unit 1)
 				)
@@
 	)
 	(symbol
-		(lib_id "Device:R_US")
-		(at 410.21 81.28 0)
-		(unit 1)
-		(exclude_from_sim no)
-		(in_bom yes)
-		(on_board yes)
-		(dnp no)
-		(property "Reference" "R3"
-			(at 412.75 80.0099 0)
-			(effects
-				(font
-					(size 1.27 1.27)
-				)
-				(justify left)
-			)
-		)
-		(property "Value" "1.24k"
-			(at 412.75 82.5499 0)
-			(effects
-				(font
-					(size 1.27 1.27)
-				)
-				(justify left)
-			)
-		)
-		(property "Footprint" "Resistor_SMD:R_1206_3216Metric_Pad1.30x1.75mm_HandSolder"
-			(at 411.226 81.534 90)
-			(effects
-				(font
-					(size 1.27 1.27)
-				)
-				(hide yes)
-			)
-		)
-		(property "Datasheet" "~"
-			(at 410.21 81.28 0)
-			(effects
-				(font
-					(size 1.27 1.27)
-				)
-				(hide yes)
-			)
-		)
-		(property "Description" "Resistor, US symbol"
-			(at 410.21 81.28 0)
-			(effects
-				(font
-					(size 1.27 1.27)
-				)
-				(hide yes)
-			)
-		)
-		(pin "2"
-		)
-		(pin "1"
-		)
-		(instances
-			(project "oshe_dmm_project_v1"
-				(path "/24c8480a-c336-4df0-8536-7016ee8fc0ac"
-					(reference "R3")
-					(unit 1)
-				)
-			)
-		)
-	)
-	(symbol
 		(lib_id "MCU_Microchip_ATmega:ATmega328P-A")
 		(at 58.42 72.39 0)
@@
 		(dnp no)
 		(fields_autoplaced yes)
-		(property "Reference" "R6"
+		(property "Reference" "R5"
 			(at 463.55 80.0099 0)
 			(effects
@@
 			(project "oshe_dmm_project_v1"
 				(path "/24c8480a-c336-4df0-8536-7016ee8fc0ac"
-					(reference "R6")
+					(reference "R5")
 					(unit 1)
 				)
@@
 			)
 		)
-		(property "Footprint" "Connector_USB:USB_C_Receptacle_Molex_105450-0101"
+		(property "Footprint" "Connector_USB:USB_C_Receptacle_GCT_USB4085"
 			(at 351.79 48.26 0)
 			(effects
@@
 		(dnp no)
 		(fields_autoplaced yes)
-		(property "Reference" "R9"
+		(property "Reference" "R8"
 			(at 534.67 105.4099 0)
 			(effects
@@
 			(project "oshe_dmm_project_v1"
 				(path "/24c8480a-c336-4df0-8536-7016ee8fc0ac"
-					(reference "R9")
+					(reference "R8")
 					(unit 1)
 				)
@@
 		(on_board yes)
 		(dnp no)
-		(property "Reference" "R7"
+		(property "Reference" "R6"
 			(at 524.002 118.11 0)
 			(effects
@@
 			(project "oshe_dmm_project_v1"
 				(path "/24c8480a-c336-4df0-8536-7016ee8fc0ac"
-					(reference "R7")
+					(reference "R6")
 					(unit 1)
 				)
@@
 		(dnp no)
 		(fields_autoplaced yes)
-		(property "Reference" "R8"
+		(property "Reference" "R7"
 			(at 527.05 44.4499 0)
 			(effects
@@
 			(project "oshe_dmm_project_v1"
 				(path "/24c8480a-c336-4df0-8536-7016ee8fc0ac"
-					(reference "R8")
+					(reference "R7")
 					(unit 1)
 				)
@@
 		(dnp no)
 		(fields_autoplaced yes)
-		(property "Reference" "R5"
+		(property "Reference" "R4"
 			(at 453.39 80.0099 0)
 			(effects
@@
 			(project "oshe_dmm_project_v1"
 				(path "/24c8480a-c336-4df0-8536-7016ee8fc0ac"
-					(reference "R5")
+					(reference "R4")
 					(unit 1)
 				)

Commit message: Changed some stuff
Other:
- added sheet Current_Measurement (Current_Measurement.kicad_sch)
- added sheet Input_Protection (Input_Protection.kicad_sch)
- added sheet Voltage_Measurement (Voltage_Measurement.kicad_sch)
Changed lines of the file:
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@@
+		)
+	)
+	(sheet
+		(at 17.78 350.52)
+		(size 40.64 16.51)
+		(fields_autoplaced yes)
+		(stroke
+			(width 0.1524)
+			(type solid)
+		)
+		(fill
+			(color 0 0 0 0.0000)
+		)
+		(property "Sheetname" "Current_Measurement"
+			(at 17.78 349.8084 0)
+			(effects
+				(font
+					(size 1.27 1.27)
+				)
+				(justify left bottom)
+			)
+		)
+		(property "Sheetfile" "Current_Measurement.kicad_sch"
+			(at 17.78 367.6146 0)
+			(effects
+				(font
+					(size 1.27 1.27)
+				)
+				(justify left top)
+			)
+		)
+		(instances
+			(project "oshe_dmm_project_v1"
+				(path "/24c8480a-c336-4df0-8536-7016ee8fc0ac"
+					(page "3")
+				)
+			)
+		)
+	)
+	(sheet
+		(at 62.23 378.46)
+		(size 38.1 20.32)
+		(fields_autoplaced yes)
+		(stroke
+			(width 0.1524)
+			(type solid)
+		)
+		(fill
+			(color 0 0 0 0.0000)
+		)
+		(property "Sheetname" "Input_Protection"
+			(at 62.23 377.7484 0)
+			(effects
+				(font
+					(size 1.27 1.27)
+				)
+				(justify left bottom)
+			)
+		)
+		(property "Sheetfile" "Input_Protection.kicad_sch"
+			(at 62.23 399.3646 0)
+			(effects
+				(font
+					(size 1.27 1.27)
+				)
+				(justify left top)
+			)
+		)
+		(instances
+			(project "oshe_dmm_project_v1"
+				(path "/24c8480a-c336-4df0-8536-7016ee8fc0ac"
+					(page "4")
+				)
+			)
+		)
+	)
+	(sheet
+		(at 17.78 378.46)
+		(size 40.64 20.32)
+		(fields_autoplaced yes)
+		(stroke
+			(width 0.1524)
+			(type solid)
+		)
+		(fill
+			(color 0 0 0 0.0000)
+		)
+		(property "Sheetname" "Voltage_Measurement"
+			(at 17.78 377.7484 0)
+			(effects
+				(font
+					(size 1.27 1.27)
+				)
+				(justify left bottom)
+			)
+		)
+		(property "Sheetfile" "Voltage_Measurement.kicad_sch"
+			(at 17.78 399.3646 0)
+			(effects
+				(font
+					(size 1.27 1.27)
+				)
+				(justify left top)
+			)
+		)
+		(instances
+			(project "oshe_dmm_project_v1"
+				(path "/24c8480a-c336-4df0-8536-7016ee8fc0ac"
+					(page "2")
+				)
+			)
 		)
 	)

Commit message: Made changes to PCB and Schematic
Parts:
- removed D2: PGOOD, LED_SMD:LED_1206_3216Metric_Pad1.42x1.75mm_HandSolder, symbol Device:LED
- removed R7: 1.5k, Resistor_SMD:R_1206_3216Metric_Pad1.30x1.75mm_HandSolder, symbol Device:R_US
- added TP1: TestPoint, TestPoint:TestPoint_Keystone_5019_Minature, symbol Connector:TestPoint
- C11: value 1.0uF -> 1uF; footprint Capacitor_SMD:C_1206_3216Metric_Pad1.33x1.80mm_HandSolder -> Capacitor_SMD:CP_Elec_4x4.5
- C8: value 0.1uF -> 1uF; footprint Capacitor_SMD:C_1206_3216Metric_Pad1.33x1.80mm_HandSolder -> Capacitor_SMD:CP_Elec_4x4.5
- R3: value 49.9k -> 10k
- R4: value 1.07k -> 1.5k
- R5: value 750 -> 1.78k
- renumbered D3 to D2, D4 to D3, R9 to R7
Connections:
- net 9V_BAT_IN: now also U2.5 (EN2)
- net TS: now also R3.1
- net USB_Power_IN: no longer U2.5 (EN2)
- net at U2.7 (~{PGOOD}): now also TP1.1
- net R-TMR: no longer names the net of U2.14 (TMR)
- net R-TMR: no longer R3.1
- no-connect marks 0 -> 1
Other:
- moved on the sheet: BAT+1, BAT-1, C6, C7, C9, D2, J2, JP1, R4, R5, R7, SW2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
