File: oshe_dmm_KiCAD/oshe_dmm_project_v1/oshe_dmm_project_v1.kicad_sch (KiCad schematic)
At the start: 37 parts, among them J1 FTDI Basic, J2 USB_C_Receptacle_USB2.0_14P, SW1 SW_Push, SW2 Power_Switch, U1 ATmega328P-A, U2 BQ24075RGT, U3 LM317_SOT-223, Y1 16MHz

Commit message: Worked on the PCB
Parts:
- added C2: 0.1uF, Capacitor_SMD:C_1206_3216Metric_Pad1.33x1.80mm_HandSolder, symbol Device:C
- added R1: 0.064, Resistor_SMD:R_2512_6332Metric_Pad1.40x3.35mm_HandSolder, symbol Device:R_US
- added R2, R3: 1k, Resistor_SMD:R_1206_3216Metric_Pad1.30x1.75mm_HandSolder, symbol Device:R_US
- added R7: 0, Resistor_SMD:R_1206_3216Metric_Pad1.30x1.75mm_HandSolder, symbol Device:R_US
- added TP1, TP2: TestPoint, TestPoint:TestPoint_Keystone_5019_Minature, symbol Connector:TestPoint
- added U2: INA219BxD, Package_SO:SOIC-8_3.9x4.9mm_P1.27mm, symbol Sensor_Energy:INA219BxD
- renumbered C9 to C10, C10 to C11, C11 to C12, C2 to C3, C3 to C4, C4 to C5, C5 to C6, C6 to C7, C7 to C8, C8 to C9, R6 to R10, R7 to R11, R8 to R12, R1 to R4, R2 to R5, R3 to R6, R4 to R8, R5 to R9, TP1 to TP3, U2 to U3, U3 to U4
Connections:
- net +5V: now also C2.2, U2.5 (VS)
- net GND: now also C2.1, R2.1, R3.1, R7.2, TP2.1, U2.6 (GND)
- net SCL: now also U2.4 (SCL)
- net SDA: now also U2.3 (SDA)
- net at BAT+1.1, C7.1, JP1.2 (C): now also TP1.1
- net at U3.14 (TMR): now also R7.1
- new net: R3.2, U2.1 (A1)
- new net: R2.2, U2.2 (A0)
- new net Current Negative: R1.2, U2.7 (IN-)
- new net Current Positive: R1.1, U2.8 (IN+)
- no-connect marks 1 -> 0
Other:
- removed sheet Current_Measurement
- note added: "Current Measurement (INA219B)"
- moved on the sheet: C7, JP1, JP2, R6, R8, SW2, Thermistor1

Commit message: PCB Design Work
Parts:
- removed SW2: Power_Switch, Button_Switch_SMD:SW_SPDT_CK_JS102011SAQN, symbol Switch:SW_SPST
- added J3: Conn_01x02, Connector_PinHeader_2.54mm:PinHeader_1x02_P2.54mm_Vertical, symbol Connector_Generic:Conn_01x02
- added TP3, TP4: TestPoint, TestPoint:TestPoint_Keystone_5019_Minature, symbol Connector:TestPoint
- renumbered TP3 to TP5
Connections:
- net +5V: now also TP3.1
- net 9V_BAT_IN: now also J3.1 (Pin_1), TP4.1
- net at JP2.2 (C): now also J3.2 (Pin_2)
Changed lines of the file:
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@@
 	)
 	(junction
+		(at 502.92 38.1)
+		(diameter 0)
+		(color 0 0 0 0)
+	)
+	(junction
 		(at 436.88 83.82)
 		(diameter 0)
@@
 	)
 	(junction
+		(at 480.06 120.65)
+		(diameter 0)
+		(color 0 0 0 0)
+	)
+	(junction
 		(at 542.29 100.33)
 		(diameter 0)
@@
 	(wire
 		(pts
-			(xy 527.05 38.1) (xy 537.21 38.1)
+			(xy 73.66 69.85) (xy 77.47 69.85)
 		)
 		(stroke
@@
 	(wire
 		(pts
-			(xy 73.66 69.85) (xy 77.47 69.85)
+			(xy 95.25 39.37) (xy 99.06 39.37)
 		)
 		(stroke
@@
 	(wire
 		(pts
-			(xy 95.25 39.37) (xy 99.06 39.37)
+			(xy 44.45 161.29) (xy 48.26 161.29)
 		)
 		(stroke
@@
 	(wire
 		(pts
-			(xy 44.45 161.29) (xy 48.26 161.29)
+			(xy 458.47 110.49) (xy 466.09 110.49)
 		)
 		(stroke
@@
 	(wire
 		(pts
-			(xy 458.47 110.49) (xy 462.28 110.49)
+			(xy 521.97 113.03) (xy 521.97 115.57)
 		)
 		(stroke
@@
 	(wire
 		(pts
-			(xy 521.97 113.03) (xy 521.97 115.57)
+			(xy 468.63 110.49) (xy 468.63 109.22)
 		)
 		(stroke
@@
 	(wire
 		(pts
+			(xy 466.09 110.49) (xy 466.09 109.22)
+		)
+		(stroke
+			(width 0)
+			(type default)
+		)
+	)
+	(wire
+		(pts
 			(xy 532.13 100.33) (xy 542.29 100.33)
 		)
@@
 	(wire
 		(pts
+			(xy 502.92 35.56) (xy 502.92 38.1)
+		)
+		(stroke
+			(width 0)
+			(type default)
+		)
+	)
+	(wire
+		(pts
 			(xy 452.12 81.28) (xy 452.12 83.82)
 		)
@@
 	(wire
 		(pts
-			(xy 476.25 110.49) (xy 472.44 110.49)
-		)
-		(stroke
-			(width 0)
-			(type default)
-		)
-	)
-	(wire
-		(pts
 			(xy 373.38 115.57) (xy 387.35 115.57)
 		)
@@
 	(wire
 		(pts
-			(xy 553.72 100.33) (xy 560.07 100.33)
+			(xy 553.72 100.33) (xy 561.34 100.33)
+		)
+		(stroke
+			(width 0)
+			(type default)
+		)
+	)
+	(wire
+		(pts
+			(xy 468.63 110.49) (xy 476.25 110.49)
 		)
 		(stroke
@@
 	(wire
 		(pts
+			(xy 527.05 38.1) (xy 537.21 38.1)
+		)
+		(stroke
+			(width 0)
+			(type default)
+		)
+	)
+	(wire
+		(pts
 			(xy 461.01 83.82) (xy 477.52 83.82)
 		)
@@
 	(wire
 		(pts
+			(xy 480.06 120.65) (xy 480.06 124.46)
+		)
+		(stroke
+			(width 0)
+			(type default)
+		)
+	)
+	(wire
+		(pts
 			(xy 31.75 88.9) (xy 34.29 88.9)
 		)
@@
 	(global_label "+5V"
 		(shape output)
-		(at 560.07 100.33 0)
+		(at 561.34 100.33 0)
 		(fields_autoplaced yes)
 		(effects
@@
 		)
 		(property "Intersheetrefs" "${INTERSHEET_REFS}"
-			(at 566.9257 100.33 0)
+			(at 568.1957 100.33 0)
 			(effects
 				(font
@@
 	)
 	(symbol
+		(lib_id "Connector:TestPoint")
+		(at 480.06 124.46 0)
+		(mirror x)
+		(unit 1)
+		(exclude_from_sim no)
+		(in_bom yes)
+		(on_board yes)
+		(dnp no)
+		(property "Reference" "TP3"
+			(at 482.6 129.0321 0)
+			(effects
+				(font
+					(size 1.27 1.27)
+				)
+				(justify left)
+			)
+		)
+		(property "Value" "TestPoint"
+			(at 482.6 126.4921 0)
+			(effects
+				(font
+					(size 1.27 1.27)
+				)
+				(justify left)
+			)
+		)
+		(property "Footprint" "TestPoint:TestPoint_Keystone_5019_Minature"
+			(at 485.14 124.46 0)
+			(effects
+				(font
+					(size 1.27 1.27)
+				)
+				(hide yes)
+			)
+		)
+		(property "Datasheet" "~"
+			(at 485.14 124.46 0)
+			(effects
+				(font
+					(size 1.27 1.27)
+				)
+				(hide yes)
+			)
+		)
+		(property "Description" "test point"
+			(at 480.06 124.46 0)
+			(effects
+				(font
+					(size 1.27 1.27)
+				)
+				(hide yes)
+			)
+		)
+		(pin "1"
+		)
+		(instances
+			(project "oshe_dmm_project_v1"
+				(path "/24c8480a-c336-4df0-8536-7016ee8fc0ac"
+					(reference "TP3")
+					(unit 1)
+				)
+			)
+		)
+	)
+	(symbol
 		(lib_id "MCU_Microchip_ATmega:ATmega328P-A")
 		(at 58.42 72.39 0)
@@
 	)
 	(symbol
-		(lib_id "Switch:SW_SPST")
-		(at 467.36 110.49 0)
-		(unit 1)
-		(exclude_from_sim no)
-		(in_bom yes)
-		(on_board yes)
-		(dnp no)
-		(fields_autoplaced yes)
-		(property "Reference" "SW2"
-			(at 467.36 104.14 0)
-			(effects
-				(font
-					(size 1.27 1.27)
-				)
-			)
-		)
-		(property "Value" "Power_Switch"
-			(at 467.36 106.68 0)
-			(effects
-				(font
-					(size 1.27 1.27)
-				)
-			)
-		)
-		(property "Footprint" "Button_Switch_SMD:SW_SPDT_CK_JS102011SAQN"
-			(at 467.36 110.49 0)
-			(effects
-				(font
-					(size 1.27 1.27)
-				)
-				(hide yes)
-			)
-		)
-		(property "Datasheet" "~"
-			(at 467.36 110.49 0)
-			(effects
-				(font
-					(size 1.27 1.27)
-				)
-				(hide yes)
-			)
-		)
-		(property "Description" "Single Pole Single Throw (SPST) switch"
-			(at 467.36 110.49 0)
-			(effects
-				(font
-					(size 1.27 1.27)
-				)
-				(hide yes)
-			)
-		)
-		(pin "2"
-		)
-		(pin "1"
-		)
-		(instances
-			(project "oshe_dmm_project_v1"
-				(path "/24c8480a-c336-4df0-8536-7016ee8fc0ac"
-					(reference "SW2")
-					(unit 1)
-				)
-			)
-		)
-	)
-	(symbol
 		(lib_id "Device:R_US")
 		(at 48.26 157.48 0)
@@
 		(on_board yes)
 		(dnp no)
-		(property "Reference" "TP3"
+		(property "Reference" "TP5"
 			(at 505.46 58.9279 0)
 			(effects
@@
 			(project ""
 				(path "/24c8480a-c336-4df0-8536-7016ee8fc0ac"
-					(reference "TP3")
+					(reference "TP5")
 					(unit 1)
 				)
@@
 	)
 	(symbol
+		(lib_id "Connector_Generic:Conn_01x02")
+		(at 466.09 104.14 90)
+		(unit 1)
+		(exclude_from_sim no)
+		(in_bom yes)
+		(on_board yes)
+		(dnp no)
+		(property "Reference" "J3"
+			(at 464.82 98.806 90)
+			(effects
+				(font
+					(size 1.27 1.27)
+				)
+				(justify right)
+			)
+		)
+		(property "Value" "Conn_01x02"
+			(at 464.82 101.346 90)
+			(effects
+				(font
+					(size 1.27 1.27)
+				)
+				(justify right)
+			)
+		)
+		(property "Footprint" "Connector_PinHeader_2.54mm:PinHeader_1x02_P2.54mm_Vertical"
+			(at 466.09 104.14 0)
+			(effects
+				(font
+					(size 1.27 1.27)
+				)
+				(hide yes)
+			)
+		)
+		(property "Datasheet" "~"
+			(at 466.09 104.14 0)
+			(effects
+				(font
+					(size 1.27 1.27)
+				)
+				(hide yes)
+			)
+		)
+		(property "Description" "Generic connector, single row, 01x02, script generated (kicad-library-utils/schlib/autogen/connector/)"
+			(at 466.09 104.14 0)
+			(effects
+				(font
+					(size 1.27 1.27)
+				)
+				(hide yes)
+			)
+		)
+		(pin "2"
+		)
+		(pin "1"
+		)
+		(instances
+			(project ""
+				(path "/24c8480a-c336-4df0-8536-7016ee8fc0ac"
+					(reference "J3")
+					(unit 1)
+				)
+			)
+		)
+	)
+	(symbol
 		(lib_id "Jumper:SolderJumper_3_Open")
 		(at 480.06 110.49 270)
@@
 					(unit 1)
 				)
+			)
+		)
+	)
+	(symbol
+		(lib_id "Connector:TestPoint")
+		(at 502.92 35.56 0)
+		(unit 1)
+		(exclude_from_sim no)
+		(in_bom yes)
+		(on_board yes)
+		(dnp no)
+		(property "Reference" "TP4"
+			(at 505.46 30.9879 0)
+			(effects
+				(font
+					(size 1.27 1.27)
+				)
+				(justify left)
+			)
+		)
+		(property "Value" "TestPoint"
+			(at 505.46 33.5279 0)
+			(effects
+				(font
+					(size 1.27 1.27)
+				)
+				(justify left)
+			)
+		)
+		(property "Footprint" "TestPoint:TestPoint_Keystone_5019_Minature"
+			(at 508 35.56 0)
+			(effects
+				(font
+					(size 1.27 1.27)
+				)
+				(hide yes)
+			)
+		)
+		(property "Datasheet" "~"
+			(at 508 35.56 0)
+			(effects
+				(font
+					(size 1.27 1.27)
+				)
+				(hide yes)
+			)
+		)
+		(property "Description" "test point"
+			(at 502.92 35.56 0)
+			(effects
+				(font
+					(size 1.27 1.27)
+				)
+				(hide yes)
+			)
+		)
+		(pin "1"
+		)
+		(instances
+			(project "oshe_dmm_project_v1"
+				(path "/24c8480a-c336-4df0-8536-7016ee8fc0ac"
+					(reference "TP4")
+					(unit 1)
+				)

Commit message: Made some more PCB changes
Parts:
- removed J2: USB_C_Receptacle_USB2.0_14P, Connector_USB:USB_C_Receptacle_GCT_USB4085, symbol Connector:USB_C_Receptacle_USB2.0_14P
- removed JP3: SolderJumper_2_Open, Jumper:SolderJumper-2_P1.3mm_Open_Pad1.0x1.5mm, symbol Jumper:SolderJumper_2_Open
- added J2: USB_C_Receptacle_PowerOnly_6P, Connector_USB:USB_C_Receptacle_GCT_USB4125-xx-x-0190_6P_TopMnt_Horizontal, symbol Connector:USB_C_Receptacle_PowerOnly_6P
- Y1: footprint Crystal:Resonator_Murata_CSTLSxxxG-3Pin_W8.0mm_H3.0mm -> Crystal:Crystal_HC49-U_Vertical
- renumbered TP3 to 5V, TP1 to BAT, TP4 to BMS_Out, TP2 to GND, TP5 to PGOOD
Connections:
- net GND: now also J2.A12 (GND), J2.B12 (GND), J2.S1 (SHIELD)
- net USB_Power_IN: now also J2.A9 (VBUS), J2.B9 (VBUS)
- no-connect marks 0 -> 2
Other:
- moved on the sheet: C8
