File: oshe_dmm_KiCAD/oshe_dmm_project_v1/oshe_dmm_project_v1.kicad_pcb (KiCad board)
At the start: 2 copper layers, 91.9 x 127.5 mm, 40 parts, among them J1 FTDI Basic, J2 USB_C_Receptacle_USB2.0_14P, SW1 SW_Push, SW2 SW_SPST, U1 ATmega328P-A, U2 BQ24075RGT, U3 LM317_SOT-223, Y1 16MHz

Commit message: Made some changes to the PCB
Parts:
- SW2: value SW_SPST -> Power_Switch; footprint Button_Switch_SMD:SW_SPST_B3S-1000 -> Button_Switch_SMD:SW_SPDT_CK_JS102011SAQN
- moved C7 85.5 mm to (74.7, 150.4), turned to 90 degrees
- moved J2 82.7 mm to (65.0, 150.4), turned to -90 degrees
- moved SW2 66.8 mm to (150.4, 150.4), turned to 90 degrees
- moved C8 60.4 mm to (93.9, 135.6), turned to -90 degrees
- moved JP2 55.6 mm to (141.2, 150.6), turned to 90 degrees
- moved JP1 49.9 mm to (76.2, 123.4), turned to -90 degrees
- moved C9 47.9 mm to (123.5, 114.3), turned to 180 degrees
- moved BAT-1 47.6 mm to (67.1, 135.1)
- moved C11 47.3 mm to (138.8, 110.2), turned to 90 degrees
- moved C6 45.3 mm to (72.1, 125.0), turned to -90 degrees
- moved BAT+1 42.8 mm to (67.1, 123.0)
- moved R4 42.2 mm to (89.4, 120.9)
- moved R5 42.2 mm to (89.4, 124.2)
- moved R6 42.2 mm to (89.4, 127.5)
- moved R3 41.9 mm to (89.4, 117.3)
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- renumbered C9 to C8, C8 to C9
Other:
- copper layers 2 -> 4

Commit message: Made more PCB changes
Parts:
- removed the D3 at (128.1, 97.3)
- removed D5: 1N4002, Diode_THT:D_DO-41_SOD81_P10.16mm_Horizontal
- added D4: 1N4002, Diode_SMD:D_1206_3216Metric_Pad1.42x1.75mm_HandSolder, F.Cu at (190.9, 211.5)
- BAT+1, BAT-1, Thermistor1: footprint TestPoint:TestPoint_Pad_4.0x4.0mm -> TestPoint:TestPoint_THTPad_D4.0mm_Drill2.0mm
- C10: value C -> 10uF
- R7: value ? -> 1.2k
- R9: value 240 -> 390
- moved C10 125.2 mm to (182.3, 211.0), turned to 90 degrees
- moved C11 124.4 mm to (198.0, 219.6), turned to -90 degrees
- moved R9 124.2 mm to (182.3, 216.6)
- moved R7 124.0 mm to (185.8, 211.0), turned to 90 degrees
- moved U3 120.8 mm to (188.9, 218.1)
- moved C8 116.6 mm to (175.7, 218.6), turned to 90 degrees
- moved JP3 111.8 mm to (197.5, 211.0), turned to -90 degrees
- moved D2 107.2 mm to (157.6, 217.1)
- moved R3 107.2 mm to (143.4, 210.0)
- moved R5 107.2 mm to (143.4, 216.9)
- moved R6 107.2 mm to (143.4, 220.2)
- moved R8 107.2 mm to (152.0, 217.1)
- moved C9 107.2 mm to (147.9, 228.3)
- moved D3 107.2 mm to (157.6, 220.7)
- moved R10 107.2 mm to (152.0, 220.7)
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- renumbered C5 to C3, C3 to C4, C4 to C5, C9 to C8, C8 to C9, D4 to D3
Other:
- board size 91.9 x 127.5 mm -> 101.6 x 177.8 mm

Commit message: Made more changes
Parts:
- removed the R3 at (143.4, 210.0)
- J2: footprint Connector_USB:USB_C_Receptacle_Molex_105450-0101 -> Connector_USB:USB_C_Receptacle_GCT_USB4085
- moved J2 4.99 mm to (122.6, 222.0)
- renumbered R4 to R3, R5 to R4, R6 to R5, R7 to R6, R8 to R7, R9 to R8, R10 to R9
Connections:
- U2 pad 15: /R-ITERM -> GND

Commit message: Made changes to PCB and Schematic
Parts:
- removed D4: 1N4002, Diode_SMD:D_1206_3216Metric_Pad1.42x1.75mm_HandSolder
- added C12: 0.1uF, Capacitor_SMD:C_0201_0603Metric_Pad0.64x0.40mm_HandSolder, F.Cu at (169.9, 131.2)
- added R10: 1k, Resistor_SMD:R_0603_1608Metric_Pad0.98x0.95mm_HandSolder, F.Cu at (170.1, 136.5)
- added R11: 1K, Resistor_SMD:R_0603_1608Metric_Pad0.98x0.95mm_HandSolder, F.Cu at (170.1, 139.0)
- added TP1: TestPoint, TestPoint:TestPoint_Keystone_5019_Minature, F.Cu at (134.0, 183.1)
- added U4: INA219BxD, Package_SO:SOIC-8_3.9x4.9mm_P1.27mm, F.Cu at (163.7, 138.6)
- C11: value 1.0uF -> 1uF; footprint Capacitor_SMD:C_1206_3216Metric_Pad1.33x1.80mm_HandSolder -> Capacitor_SMD:CP_Elec_4x4.5
- C8: value 0.1uF -> 1uF; footprint Capacitor_SMD:C_1206_3216Metric_Pad1.33x1.80mm_HandSolder -> Capacitor_SMD:CP_Elec_4x4.5
- D2: value PGOOD -> CHG
- D3: value CHG -> 1N4002; footprint LED_SMD:LED_1206_3216Metric_Pad1.42x1.75mm_HandSolder -> Diode_SMD:D_1206_3216Metric_Pad1.42x1.75mm_HandSolder
- R3: value 49.9k -> 10k
- R4: value 1.07k -> 1.5k
- R5: value 750 -> 1.78k
- R9: value 1.5k -> 0.064; footprint Resistor_SMD:R_1206_3216Metric_Pad1.30x1.75mm_HandSolder -> Resistor_SMD:R_2512_6332Metric_Pad1.40x3.35mm_HandSolder
- moved SW2 98.8 mm to (115.7, 208.5), turned to -90 degrees
- moved R9 88.7 mm to (164.0, 132.8)
- moved JP2 81.0 mm to (124.9, 208.5), turned to -90 degrees
- moved JP3 74.7 mm to (127.6, 184.7), turned to 0 degrees
- moved C11 58.9 mm to (139.1, 218.6), turned to 0 degrees
- moved U3 56.6 mm to (132.5, 213.0), turned to -90 degrees
- moved R8 49.7 mm to (133.5, 206.9), turned to 0 degrees
- moved R6 46.8 mm to (139.1, 209.5), turned to 0 degrees
- moved BAT-1 46.0 mm to (159.5, 235.9), turned to 180 degrees
- moved C8 46.0 mm to (132.5, 202.9), turned to 0 degrees
- moved BAT+1 45.4 mm to (146.2, 235.9), turned to 180 degrees
- moved Thermistor1 44.6 mm to (152.8, 235.9)
- moved C10 43.4 mm to (139.1, 206.9), turned to 0 degrees
- moved C6 41.0 mm to (152.3, 230.8), turned to 0 degrees
- moved C7 39.3 mm to (140.2, 187.5), turned to 0 degrees
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Connections:
- C10 pad 1: Net-(D4-A) -> Net-(D3-A)
- D3 pad 1: Net-(D3-K) -> +5V
- R3 pad 1: /R-TMR -> TS
- R6 pad 1: Net-(D4-A) -> Net-(D3-A)
- R8 pad 2: Net-(D4-A) -> Net-(D3-A)
- R9 pad 1: 9V_BAT_IN -> Current Positive
- R9 pad 2: Net-(D3-A) -> Current Negative
- U2 pad 14: /R-TMR -> unconnected-(U2-TMR-Pad14)
- U2 pad 5: USB_Power_IN -> 9V_BAT_IN
- U2 pad 7: Net-(D2-K) -> Net-(U2-~{PGOOD})
- U2 pad 9: Net-(D3-K) -> Net-(D2-K)
- U3 pad 1: Net-(D4-A) -> Net-(D3-A)
Routing:
- net Net-(JP1-C): track 0.00 -> 11.5 mm
- net TS: track 0.00 -> 8.86 mm
- added copper zone on F.Cu, net GND
Other:
- board text added: "Battery System"
- board text added: "Inputs & Input Protection?"

Commit message: Made some PCB changes
Parts:
- moved SW2 97.6 mm to (213.3, 211.6), turned to 90 degrees
- moved JP3 94.1 mm to (207.8, 234.0), turned to 180 degrees
- moved J2 91.8 mm to (209.2, 199.9), turned to 90 degrees
- moved U2 87.5 mm to (208.4, 225.2), turned to 180 degrees
- moved TP1 85.5 mm to (201.4, 235.6), turned to 180 degrees
- moved R4 80.8 mm to (201.4, 231.6), turned to 180 degrees
- moved JP2 79.3 mm to (204.1, 211.6), turned to 90 degrees
- moved R5 77.3 mm to (201.4, 228.3), turned to 180 degrees
- moved R7 73.9 mm to (201.4, 224.5), turned to 180 degrees
- moved C7 70.2 mm to (195.2, 231.2), turned to 180 degrees
- moved C9 66.2 mm to (195.2, 227.8), turned to 180 degrees
- moved C8 65.6 mm to (196.5, 217.2), turned to 180 degrees
- moved U3 64.3 mm to (196.5, 207.1), turned to 90 degrees
- moved D2 62.9 mm to (195.3, 224.5), turned to 180 degrees
- moved R8 62.3 mm to (195.5, 213.2), turned to 180 degrees
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
Commit message: Worked on the PCB
Parts:
- removed the C12 at (169.9, 131.2)
- removed the R10 at (170.1, 136.5)
- removed the R11 at (170.1, 139.0)
- removed the R9 at (164.0, 132.8)
- removed the U4 at (163.7, 138.6)
- added C2: 0.1uF, Capacitor_SMD:C_1206_3216Metric_Pad1.33x1.80mm_HandSolder, F.Cu at (119.8, 195.8)
- added R1: 0.064, Resistor_SMD:R_2512_6332Metric_Pad1.40x3.35mm_HandSolder, F.Cu at (122.2, 200.1)
- added R2: 1k, Resistor_SMD:R_1206_3216Metric_Pad1.30x1.75mm_HandSolder, F.Cu at (122.6, 183.7)
- added R3: 1k, Resistor_SMD:R_1206_3216Metric_Pad1.30x1.75mm_HandSolder, F.Cu at (125.0, 183.7)
- added R7: 0, Resistor_SMD:R_1206_3216Metric_Pad1.30x1.75mm_HandSolder, F.Cu at (172.7, 219.5)
- added TP1: TestPoint, TestPoint:TestPoint_Keystone_5019_Minature, F.Cu at (183.8, 230.8)
- added TP2: TestPoint, TestPoint:TestPoint_Keystone_5019_Minature, F.Cu at (170.2, 230.4)
- added U2: INA219BxD, Package_SO:SOIC-8_3.9x4.9mm_P1.27mm, F.Cu at (121.9, 190.7)
- D2: moved to B.Cu
- R11: renamed from R7; moved to B.Cu
- moved C12 32.7 mm to (193.4, 234.0), turned to -90 degrees
- moved C8 32.2 mm to (202.8, 199.8), turned to -90 degrees
- moved U3 31.2 mm to (177.7, 219.9), turned to 90 degrees
- moved R8 31.1 mm to (174.1, 216.6)
- moved R9 29.3 mm to (172.7, 222.1)
- moved JP3 28.8 mm to (206.5, 205.3), turned to -90 degrees
- moved D3 26.9 mm to (198.5, 232.5), turned to 0 degrees
- moved R10 26.5 mm to (202.5, 234.0), turned to -90 degrees
- moved C11 26.1 mm to (205.1, 234.4), turned to -90 degrees
- moved C10 25.1 mm to (174.1, 214.1)
- moved TP3 24.4 mm to (183.2, 219.4)
- moved U4 20.5 mm to (199.0, 227.4), turned to 180 degrees
- moved R12 18.5 mm to (205.1, 228.9), turned to -90 degrees
- moved C9 16.3 mm to (209.2, 227.4), turned to -90 degrees
- moved D2 15.8 mm to (211.0, 223.1), turned to 0 degrees
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- renumbered C9 to C10, C10 to C11, C11 to C12, C2 to C3, C3 to C4, C4 to C5, C5 to C6, C6 to C7, C7 to C8, C8 to C9, R6 to R10, R8 to R12, R1 to R4, R2 to R5, R3 to R6, R4 to R8, R5 to R9, TP1 to TP3, U2 to U3, U3 to U4
Connections:
- U3 pad 14: unconnected-(U2-TMR-Pad14) -> Net-(U3-TMR)
Routing:
- net 9V_BAT_IN: track 0.00 -> 52.2 mm, vias 0 -> 1
- net Net-(D2-K): track 0.00 -> 34.4 mm, vias 0 -> 1
- net Net-(JP1-C): track 11.5 -> 0.00 mm
- net USB_Power_IN: track 0.00 -> 8.67 mm
- net Net-(JP2-C): track 0.00 -> 7.29 mm
- net TS: track 8.86 -> 16.0 mm
- net GND: track 0.00 -> 6.76 mm, vias 0 -> 18
- net Net-(U3-~{PGOOD}): track 0.00 -> 4.13 mm
- net Net-(D2-A): track 0.00 -> 3.79 mm
- net +5V: track 0.00 -> 3.30 mm
- net /R-ILIM: track 0.00 -> 2.89 mm
- net /R-ISET: track 0.00 -> 2.87 mm
- net Net-(U3-TMR): track 0.00 -> 2.02 mm
- added copper zone on F.Cu, net +5V
- added copper zone on F.Cu, net 9V_BAT_IN
- added copper zone on F.Cu, net BMS_BAT_IN
- added copper zone on In1.Cu, net GND
- added copper zone on F.Cu, net Net-(D3-A)
- added copper zone on F.Cu, net Net-(JP1-C)
- added copper zone on F.Cu, net Net-(JP2-B)
Other:
- board text added: "BAT+1"
- board text added: "BAT-1"
- board text added: "Battery"
- board text added: "Thermistor1"

Commit message: PCB Design Work
Parts:
- removed SW2: Power_Switch, Button_Switch_SMD:SW_SPDT_CK_JS102011SAQN
- added J3: Conn_01x02, Connector_PinHeader_2.54mm:PinHeader_1x02_P2.54mm_Vertical, F.Cu at (201.2, 211.9)
- added REF** (x2): OSHW-Symbol_13.4x12mm_Copper, Symbol:OSHW-Symbol_13.4x12mm_Copper, F.Cu at (125.5, 72.3)
- added REF**: KiCad-Logo2_8mm_SilkScreen, Symbol:KiCad-Logo2_8mm_SilkScreen, F.Cu at (199.8, 72.1)
- added REF**: Symbol_HighVoltage_Triangle_17x15mm_Copper, Symbol:Symbol_HighVoltage_Triangle_17x15mm_Copper, F.Cu at (154.1, 231.7)
- added TP3: TestPoint, TestPoint:TestPoint_Keystone_5019_Minature, F.Cu at (195.1, 221.8)
- added TP4: TestPoint, TestPoint:TestPoint_Keystone_5019_Minature, F.Cu at (180.5, 213.9)
- moved SW1 97.5 mm to (119.8, 125.8), turned to 180 degrees
- moved R5 93.5 mm to (119.8, 132.4), turned to -90 degrees
- moved C5 63.2 mm to (126.0, 163.1), turned to -90 degrees
- moved C3 62.9 mm to (122.5, 152.5), turned to 180 degrees
- moved C1 59.7 mm to (125.0, 132.6), turned to -90 degrees
- moved C6 59.4 mm to (129.1, 163.1), turned to 90 degrees
- moved U1 58.6 mm to (124.5, 144.3), turned to 90 degrees
- moved D1 57.4 mm to (128.5, 127.1), turned to -90 degrees
- moved Y1 56.5 mm to (128.5, 157.0), turned to 180 degrees
- moved R4 54.8 mm to (128.5, 132.6), turned to -90 degrees
- moved C4 23.5 mm to (122.5, 119.4), turned to 180 degrees
- moved J1 18.0 mm to (120.9, 115.9), turned to 90 degrees
- moved JP2 12.0 mm to (201.2, 220.5), turned to 0 degrees
- moved J2 7.83 mm to (205.9, 207.0)
- moved JP3 7.83 mm to (198.8, 204.1)
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- renumbered TP3 to TP5
Routing:
- net USB_Power_IN: track 8.67 -> 51.6 mm
- net GND: track 6.76 -> 27.1 mm
- net unconnected-(J2-SHIELD-PadS1): track 0.00 -> 15.4 mm
- net 9V_BAT_IN: track 52.2 -> 40.3 mm
- net Current Negative: track 0.00 -> 9.46 mm
- net Current Positive: track 0.00 -> 7.50 mm
- net Net-(JP2-B): track 0.02 -> 4.72 mm
- net Net-(U2-A1): track 0.00 -> 3.84 mm
- net TS: track 16.0 -> 12.3 mm
- net +5V: track 3.30 -> 6.26 mm, vias 0 -> 12
- net Net-(U2-A0): track 0.00 -> 2.96 mm
- net Net-(U3-~{PGOOD}): track 4.13 -> 5.67 mm, vias 0 -> 2
- net Net-(J3-Pin_2): track 7.29 -> 6.10 mm
- net Net-(D2-K): track 34.4 -> 33.4 mm
- added copper zone on F.Cu, net TS
- added copper zone on F.Cu, net USB_Power_IN
Other:
- outline, holes or cut-outs redrawn
- board text added: "Designed By: Peter Kocour, Alex Ritter, Ethan Dwyer, Luc Prisby, Caleb Jahncke, James Lovell"
- board text added: "Digital Multimeter V1"
- board text added: "oshe.io"

Commit message: Made some more PCB changes
Parts:
- removed JP3: SolderJumper_2_Open, Jumper:SolderJumper-2_P1.3mm_Open_Pad1.0x1.5mm
- 5V: renamed from TP3; moved to B.Cu
- BAT: renamed from TP1; moved to B.Cu
- BMS_Out: renamed from TP4; moved to B.Cu
- GND: renamed from TP2; moved to B.Cu
- J2: value USB_C_Receptacle_USB2.0_14P -> USB_C_Receptacle_PowerOnly_6P; footprint Connector_USB:USB_C_Receptacle_GCT_USB4085 -> Connector_USB:USB_C_Receptacle_GCT_USB4125-xx-x-0190_6P_TopMnt_Horizontal
- PGOOD: renamed from TP5; moved to B.Cu
- Y1: footprint Crystal:Resonator_Murata_CSTLSxxxG-3Pin_W8.0mm_H3.0mm -> Crystal:Crystal_HC49-U_Vertical
- moved C6 77.2 mm to (51.8, 161.6), turned to 0 degrees
- moved C5 74.3 mm to (51.8, 158.6), turned to 180 degrees
- moved Y1 69.8 mm to (58.7, 157.5), turned to -90 degrees
- moved J1 61.5 mm to (69.5, 149.5)
- moved C3 57.9 mm to (64.8, 157.3), turned to 90 degrees
- moved U1 53.7 mm to (72.9, 159.3), turned to 0 degrees
- moved R4 53.6 mm to (84.6, 163.4), turned to 180 degrees
- moved D1 52.8 mm to (90.2, 163.4), turned to 180 degrees
- moved C4 49.2 mm to (91.2, 157.4), turned to 90 degrees
- moved C1 48.7 mm to (84.6, 159.8), turned to 180 degrees
- moved R5 41.5 mm to (84.9, 154.7), turned to 180 degrees
- moved C12 41.4 mm to (206.8, 194.8), turned to 90 degrees
- moved C11 41.2 mm to (195.1, 194.4), turned to 90 degrees
- moved BAT-1 39.9 mm to (210.0, 230.2), turned to -90 degrees
- moved R10 39.5 mm to (197.8, 194.8), turned to 90 degrees
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Connections:
- J2 pad S1: unconnected-(J2-SHIELD-PadS1) -> GND
Routing:
- net USB_Power_IN: track 51.6 -> 0.00 mm
- net unconnected-(J2-SHIELD-PadS1): track 15.4 -> 0.00 mm
- net Net-(U3-~{PGOOD}): track 5.67 -> 19.5 mm, vias 2 -> 1
- net 9V_BAT_IN: track 40.3 -> 32.0 mm, vias 1 -> 5
- net Net-(U3-TMR): track 2.02 -> 8.30 mm
- net Net-(JP1-C): track 0.00 -> 5.46 mm
- net Net-(D2-K): track 33.4 -> 28.2 mm
- net TS: track 12.3 -> 7.36 mm
- net Net-(JP2-B): track 4.72 -> 0.47 mm
- net GND: track 27.1 -> 22.9 mm, vias 18 -> 20
- net /R-ISET: track 2.80 -> 5.17 mm
- net +5V: track 6.26 -> 4.37 mm, vias 12 -> 11
- net Net-(D2-A): track 3.79 -> 2.33 mm
- net Net-(J3-Pin_2): track 6.10 -> 4.95 mm
- added copper zone on B.Cu, net +5V
- added copper zone on In2.Cu, net +5V
- added copper zone on B.Cu, net GND
Other:
- board text removed: "Battery"
- board text removed: "Inputs & Input Protection?"
