File: oshe_dmm_KiCAD/oshe_dmm_project_v1/Input_Protection.kicad_sch (KiCad schematic)
At the start: 0 parts

Commit message: Updated input protection schematic.
Parts:
- added C1: 0.15 μf, oshe:CKG57K, symbol Device:C
- added COMin1, Vin1: ~, symbol oshe:Input
- added D1: SMAJ200CA, Diode_SMD:D_SMA, symbol Diode:SMAJ200CA
- added F1: Fuse, symbol Device:Fuse
- added R1: R_US, symbol Device:R_US
- added R2: 10k, symbol Device:R_US
- added Vout+1, Vout-1: ~, symbol oshe:Node
Connections:
- new net: C1.2, COMin1., D1.1 (A1), Vout-1.
- new net: D1.2 (A2), R1.2, R2.1
- new net: C1.1, R2.2, Vout+1.
- new net: F1.1, Vin1.
- new net: F1.2, R1.1
