File: oshe_dmm_KiCAD/oshe_dmm_project_v1/Voltage_Measurement.kicad_sch (KiCad schematic)
At the start: 0 parts

Commit message: Update Voltage_Measurement.kicad_sch
James- copied my existing voltage circuit. This is a rough draft that contains the switch and the correct resistor values, but does NOT have the protection stuff we talked about at our last meeting. Working on that for Saturday.
Parts:
- added R1: 900K, symbol Device:R
- added R2: 90k, symbol Device:R
- added R3: 9k, symbol Device:R
- added R4: 1k, symbol Device:R
- added RV1: Varistor, symbol Device:Varistor
- added SW1: SW_Rotary_1x4_MP, symbol Switch:SW_Rotary_1x4_MP
- added TP1: V-, symbol Connector:TestPoint_Probe
- added TP2: V+, symbol Connector:TestPoint_Probe
- added U1: ADS1115IDGS, Package_SO:TSSOP-10_3x3mm_P0.5mm, symbol Analog_ADC:ADS1115IDGS
Connections:
- new net: SW1.5, U1.4 (AIN0)
- new net 200mv: R1.1, RV1.1, SW1.1, TP2.1
- new net 200v: R3.2, R4.1, SW1.4
- new net 20v: R2.2, R3.1, SW1.3
- new net 2v: R1.2, R2.1, SW1.2
- new net ground: R4.2, RV1.2, TP1.1, U1.3 (GND)

Commit message: Made some PCB and Schematic Changes
Parts:
- removed R1: 900K, symbol Device:R
- removed R2: 90k, symbol Device:R
- removed R3: 9k, symbol Device:R
- removed R4: 1k, symbol Device:R
- removed RV1: Varistor, symbol Device:Varistor
- removed SW1: SW_Rotary_1x4_MP, symbol Switch:SW_Rotary_1x4_MP
- removed TP1: V-, symbol Connector:TestPoint_Probe
- removed TP2: V+, symbol Connector:TestPoint_Probe
- removed U1: ADS1115IDGS, Package_SO:TSSOP-10_3x3mm_P0.5mm, symbol Analog_ADC:ADS1115IDGS
