File: mini_dmm/mini_dmm_KiCAD/oshe_mini_dmm_project/oshe_mini_dmm_project.kicad_pcb (KiCad board)
At the start: 2 copper layers, 1 part, among them U2 STM32F303CBTx

Commit message: Made some more updates!
Parts:
- added U1: LM324, Package_SO:SOIC-14_3.9x8.7mm_P1.27mm, F.Cu at (136.5, 96.3)
- moved U2 2.39 mm to (154.8, 96.3)

Commit message: Made some more changes
Parts:
- added BT1: Battery, Battery:BatteryHolder_Keystone_3034_1x20mm, B.Cu at (145.8, 119.4)
- added C1: 0.1uF, Capacitor_SMD:C_0805_2012Metric_Pad1.18x1.45mm_HandSolder, F.Cu at (71.1, 98.6)
- added C2: 1uF, Capacitor_SMD:C_0805_2012Metric_Pad1.18x1.45mm_HandSolder, F.Cu at (71.1, 101.6)
- added C3: 0.1uF, Capacitor_SMD:C_0805_2012Metric_Pad1.18x1.45mm_HandSolder, F.Cu at (71.1, 104.6)
- added C4: 1uF, Capacitor_SMD:C_0805_2012Metric_Pad1.18x1.45mm_HandSolder, F.Cu at (71.1, 107.6)
- added C5: 1uF, Capacitor_SMD:C_0805_2012Metric_Pad1.18x1.45mm_HandSolder, F.Cu at (71.1, 110.6)
- added C6: 0.1uF, Capacitor_SMD:C_0805_2012Metric_Pad1.18x1.45mm_HandSolder, F.Cu at (71.1, 113.6)
- added C7: 22pF, Capacitor_SMD:C_0805_2012Metric_Pad1.18x1.45mm_HandSolder, F.Cu at (129.7, 105.4)
- added C8: 22pF, Capacitor_SMD:C_0805_2012Metric_Pad1.18x1.45mm_HandSolder, F.Cu at (124.9, 105.4)
- added D1: VOLTAGE, LED_SMD:LED_0805_2012Metric_Pad1.15x1.40mm_HandSolder, F.Cu at (137.4, 75.9)
- added D2: CURRENT, LED_SMD:LED_0805_2012Metric_Pad1.15x1.40mm_HandSolder, F.Cu at (145.8, 75.9)
- added D3: RESISTANCE, LED_SMD:LED_0805_2012Metric_Pad1.15x1.40mm_HandSolder, F.Cu at (153.9, 75.9)
- added D4: NEGATIVE, LED_SMD:LED_0805_2012Metric_Pad1.15x1.40mm_HandSolder, F.Cu at (128.2, 65.3)
- added D5: Green, LED_SMD:LED_1206_3216Metric_Pad1.42x1.75mm_HandSolder, F.Cu at (154.4, 105.4)
- added F1: 500mA, Fuse:Fuse_1206_3216Metric_Pad1.42x1.75mm_HandSolder, F.Cu at (96.4, 83.4)
- added F2: 1A, Fuse:Fuse_1206_3216Metric_Pad1.42x1.75mm_HandSolder, F.Cu at (96.4, 86.7)
- added J1: FTDI Basic, Connector_PinSocket_2.54mm:PinSocket_1x06_P2.54mm_Vertical, F.Cu at (135.6, 132.6)
- added R1: 9.1MEG, Resistor_SMD:R_0805_2012Metric_Pad1.20x1.40mm_HandSolder, F.Cu at (75.8, 98.5)
- added R10: 1k, Resistor_SMD:R_0805_2012Metric_Pad1.20x1.40mm_HandSolder, F.Cu at (85.3, 98.5)
- added R11: 1k, Resistor_SMD:R_0805_2012Metric_Pad1.20x1.40mm_HandSolder, F.Cu at (85.3, 101.5)
- added R12: 1k, Resistor_SMD:R_0805_2012Metric_Pad1.20x1.40mm_HandSolder, F.Cu at (85.3, 104.4)
- added R13: 1k, Resistor_SMD:R_0805_2012Metric_Pad1.20x1.40mm_HandSolder, F.Cu at (85.3, 107.4)
- added R14: 390, Resistor_SMD:R_1206_3216Metric_Pad1.30x1.75mm_HandSolder, F.Cu at (96.4, 90.0)
- added R15: 10k, Resistor_SMD:R_1206_3216Metric_Pad1.30x1.75mm_HandSolder, F.Cu at (96.4, 93.3)
- added R2: 1MEG, Resistor_SMD:R_0805_2012Metric_Pad1.20x1.40mm_HandSolder, F.Cu at (75.8, 101.5)
- added R3: 9.1MEG, Resistor_SMD:R_0805_2012Metric_Pad1.20x1.40mm_HandSolder, F.Cu at (75.8, 104.4)
- added R4: 1MEG, Resistor_SMD:R_0805_2012Metric_Pad1.20x1.40mm_HandSolder, F.Cu at (75.8, 107.4)
- added R5: 1, Resistor_SMD:R_2512_6332Metric_Pad1.40x3.35mm_HandSolder, F.Cu at (164.1, 131.8)
- added R6: 9.1MEG, Resistor_SMD:R_0805_2012Metric_Pad1.20x1.40mm_HandSolder, F.Cu at (80.6, 98.5)
- added R7: 1MEG, Resistor_SMD:R_0805_2012Metric_Pad1.20x1.40mm_HandSolder, F.Cu at (80.6, 101.5)
- added R8: 9.1MEG, Resistor_SMD:R_0805_2012Metric_Pad1.20x1.40mm_HandSolder, F.Cu at (80.6, 104.4)
- added R9: 1MEG, Resistor_SMD:R_0805_2012Metric_Pad1.20x1.40mm_HandSolder, F.Cu at (80.6, 107.4)
- added U3: ATmega328P-A, Package_QFP:TQFP-32_7x7mm_P0.8mm, F.Cu at (127.3, 122.4)
- added U4: LM2664M6, Mini_DMM_Footprint_Library:SOT95P280X145-6N, F.Cu at (151.9, 131.6)
- added Y1: 16MHz, Crystal:Crystal_HC49-U_Vertical, F.Cu at (124.7, 110.7)
- U2: value STM32F303CBTx -> BU91796FS-ME2; footprint Package_QFP:LQFP-48_7x7mm_P0.5mm -> Mini_DMM_Footprint_Library:SSOP-A32
- moved U1 25.2 mm to (146.5, 119.4)
- moved U2 12.7 mm to (165.1, 88.9)
Connections:
- net Node_1 renamed A0
- net Node_2 renamed A1
- net Node_3 renamed A2
- net Node_4 renamed A3
- U2 pad 23: Net-(U2-VSS-Pad23) -> unconnected-(U2-VLCD-Pad23)
- U2 pad 24: unconnected-(U2-VDD-Pad24) -> +3.3V
- U2 pad 25: unconnected-(U2-PB12-Pad25) -> GND
Other:
- board outline added: 54 x 86 mm

Commit message: Made PCB updates
Parts:
- removed R14: 390, Resistor_SMD:R_1206_3216Metric_Pad1.30x1.75mm_HandSolder
- removed R15: 10k, Resistor_SMD:R_1206_3216Metric_Pad1.30x1.75mm_HandSolder
- added C10: 22pF, Capacitor_SMD:C_0805_2012Metric_Pad1.18x1.45mm_HandSolder, F.Cu at (90.6, 118.9)
- added C9: 22pF, Capacitor_SMD:C_0805_2012Metric_Pad1.18x1.45mm_HandSolder, F.Cu at (85.8, 118.9)
- added F3: 1A, Fuse:Fuse_1206_3216Metric_Pad1.42x1.75mm_HandSolder, F.Cu at (168.6, 125.5)
- added J2: TEST LEAD CONNECTIONS, Connector_PinHeader_2.54mm:PinHeader_1x06_P2.54mm_Horizontal, F.Cu at (175.3, 117.9)
- added J3: FTDI Basic, Connector_PinSocket_2.54mm:PinSocket_1x06_P2.54mm_Vertical, F.Cu at (79.5, 106.1)
- added REF** (x2): OSHW-Symbol_8.9x8mm_Copper, Symbol:OSHW-Symbol_8.9x8mm_Copper, F.Cu at (131.6, 60.7)
- added SW1: MODE SELECT, Mini_DMM_Footprint_Library:SMT_FS, F.Cu at (137.2, 89.7)
- added SW2: PTS526 SK15 SMTR2 LFS, Mini_DMM_Footprint_Library:SMT_FS, F.Cu at (105.2, 97.5)
- added SW3: SW_DPDT_x2, Mini_DMM_Footprint_Library:SW_JS102011SAQN, B.Cu at (127.3, 124.2)
- C1, C6: value 0.1uF -> 1uF
- C5: value 1uF -> 0.1uF
- C7: value 22pF -> 1uF
- C8: value 22pF -> 0.1uF
- D5: footprint LED_SMD:LED_1206_3216Metric_Pad1.42x1.75mm_HandSolder -> LED_SMD:LED_0805_2012Metric_Pad1.15x1.40mm_HandSolder
- F2: value 1A -> 500mA
- J1: value FTDI Basic -> DISPLAY; footprint Connector_PinSocket_2.54mm:PinSocket_1x06_P2.54mm_Vertical -> Mini_DMM_Footprint_Library:LCD-S401M16KR-81359
- R10: value 1k -> 300
- R12: value 1k -> 390
- R13: value 1k -> 10k
- R5: value 1 -> 0.05
- R6, R8: value 9.1MEG -> 1k
- R7, R9: value 1MEG -> 1k
- moved C2 93.6 mm to (162.9, 119.9)
- moved C1 82.2 mm to (150.4, 119.9)
- moved R11 77.4 mm to (161.3, 86.4), turned to 90 degrees
- moved R3 77.1 mm to (150.4, 124.0)
- moved R1 76.6 mm to (150.4, 115.8)
- moved R2 76.4 mm to (150.4, 117.9), turned to 180 degrees
- moved R4 76.0 mm to (150.4, 121.9), turned to 180 degrees
- moved R10 74.9 mm to (159.3, 86.4), turned to -90 degrees
- moved C6 68.1 mm to (136.1, 133.8), turned to 90 degrees
- moved F2 67.8 mm to (150.9, 127.0), turned to 180 degrees
- moved C4 64.4 mm to (130.3, 132.9), turned to -90 degrees
- moved J1 63.0 mm to (152.4, 71.9), turned to 0 degrees
- moved F1 61.8 mm to (150.9, 112.5), turned to 180 degrees
- moved D5 47.3 mm to (107.4, 111.0), turned to 180 degrees
- moved R9 34.8 mm to (103.4, 81.0), turned to 180 degrees
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Connections:
- C1 pad 2: Net-(U3-AREF) -> +3.3V
- C2 pad 1: Net-(U4-CAP+) -> -3.3V
- C2 pad 2: Net-(U4-CAP-) -> GND
- C3 pad 1: +3.3V -> GND
- C3 pad 2: GND -> Net-(U3-AREF)
- C4 pad 1: GND -> Net-(U4-CAP+)
- C4 pad 2: +3.3V -> Net-(U4-CAP-)
- C5 pad 1: GND -> +3.3V
- C5 pad 2: -3.3V -> GND
- C6 pad 1: Net-(U3-~{RESET}/PC6) -> GND
- C6 pad 2: DTR -> +3.3V
- C7 pad 1: Net-(U3-XTAL1/PB6) -> GND
- C7 pad 2: GND -> -3.3V
- C8 pad 1: GND -> Net-(U3-~{RESET}/PC6)
- C8 pad 2: Net-(U3-XTAL2/PB7) -> DTR
- F2 pad 1: LEAD_3 -> LEAD_2
- J1 pad 1: DTR -> COM0
- J1 pad 2: TXD -> COM1
- J1 pad 3: RXD -> COM2
- J1 pad 4: +3.3V -> COM3
- J1 pad 5: GND -> SEG0
- J1 pad 6: GND -> SEG1
- R10 pad 1: GND -> +3.3V
- R10 pad 2: Net-(D1-K) -> Net-(U2-VLCD)
- R11 pad 1: GND -> Net-(U2-VLCD)
- R11 pad 2: Net-(D2-K) -> GND
- R12 pad 1: GND -> Net-(D5-A)
- R12 pad 2: Net-(D3-K) -> SCK/D13
- R13 pad 1: GND -> Net-(U3-~{RESET}/PC6)
- R13 pad 2: Net-(D4-K) -> +3.3V
- R3 pad 1: LEAD_2 -> Net-(F2-Pad2)
- R5 pad 1: Net-(F2-Pad2) -> Net-(U1C-+)
- R6 pad 1: Net-(F2-Pad2) -> GND
- R6 pad 2: Net-(U1C-+) -> Net-(D1-K)
- R7 pad 1: Net-(U1C-+) -> GND
- R7 pad 2: GND -> Net-(D2-K)
- R8 pad 1: LEAD_4 -> GND
- R8 pad 2: Net-(U1D-+) -> Net-(D3-K)
- R9 pad 1: Net-(U1D-+) -> GND
- R9 pad 2: GND -> Net-(D4-K)
- U1 pad 12: Net-(U1D-+) -> LEAD_4
- U2 pad 1: unconnected-(U2-SEG_2-Pad1) -> SEG2
- U2 pad 19: unconnected-(U2-COM_0-Pad19) -> COM0
- U2 pad 2: unconnected-(U2-SEG_3-Pad2) -> SEG3
- U2 pad 20: unconnected-(U2-COM_1-Pad20) -> COM1
- U2 pad 21: unconnected-(U2-COM_2-Pad21) -> COM2
- U2 pad 22: unconnected-(U2-COM_3-Pad22) -> COM3
- U2 pad 23: unconnected-(U2-VLCD-Pad23) -> Net-(U2-VLCD)
- U2 pad 26: unconnected-(U2-TEST_1-Pad26) -> GND
- U2 pad 27: unconnected-(U2-TEST_2-Pad27) -> GND
- U2 pad 28: unconnected-(U2-OSCIN-Pad28) -> GND
- U2 pad 29: unconnected-(U2-SCL-Pad29) -> A5/SCL
- U2 pad 3: unconnected-(U2-SEG_4-Pad3) -> SEG4
- U2 pad 30: unconnected-(U2-SDA-Pad30) -> A4/SDA
- U2 pad 31: unconnected-(U2-SEG_0-Pad31) -> SEG0
- U2 pad 32: unconnected-(U2-SEG_1-Pad32) -> SEG1
- U2 pad 4: unconnected-(U2-SEG_5-Pad4) -> SEG5
- U2 pad 5: unconnected-(U2-SEG_6-Pad5) -> SEG6
- U2 pad 6: unconnected-(U2-SEG_7-Pad6) -> SEG7
Routing:
- net Net-(BT1-+): track 0.00 -> 49.0 mm
- net COM0: track 0.00 -> 31.0 mm, vias 0 -> 1
- net COM1: track 0.00 -> 29.2 mm, vias 0 -> 1
- net COM2: track 0.00 -> 27.5 mm, vias 0 -> 1
- net COM3: track 0.00 -> 25.8 mm, vias 0 -> 1
- net LEAD_1: track 0.00 -> 25.0 mm
- net LEAD_2: track 0.00 -> 24.6 mm
- net SEG7: track 0.00 -> 23.6 mm
- net GND: track 0.00 -> 23.5 mm
- net SEG6: track 0.00 -> 21.9 mm
- net SEG5: track 0.00 -> 20.4 mm
- net SEG4: track 0.00 -> 18.8 mm
- net SEG0: track 0.00 -> 18.3 mm, vias 0 -> 1
- net LEAD_4: track 0.00 -> 17.3 mm
- net SEG3: track 0.00 -> 17.1 mm
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- added copper zone on B.Cu, net +3.3V
- added copper zone on F.Cu, net +3.3V
- added copper zone on B.Cu, net -3.3V
- added copper zone on In1.Cu, net GND
- added copper zone on In2.Cu, net GND
Other:
- copper layers 2 -> 4
- board text added: "(+/-)"
- board text added: "A"
- board text added: "FUSE(1A)"
- board text added: "FUSE(500mA)"
- board text added: "Made By: Peter Kocour, Ian Ranstadler, Nathan Campbell"
- board text added: "Open Source Hardware Enterprise Mini-DMM OSHE.IO"
- board text added: "V"
- board text added: "Ω"

Commit message: PCB Updated
Parts:
- added G***: LOGO, Peter_Custom_Library:35mmX7mm_ECE_MTU, F.Cu at (159.0, 135.8)
- added G***: LOGO, Peter_Custom_Library:Calumet_Electronics_Logo_1Inch, F.Cu at (200.0, 149.0)
- moved R7 78.3 mm to (173.7, 71.3), turned to 180 degrees
- moved R8 78.3 mm to (173.7, 74.9), turned to 180 degrees
- moved R6 78.3 mm to (173.7, 67.8), turned to 180 degrees
- moved F2 72.4 mm to (222.1, 113.5)
- moved F1 71.7 mm to (222.0, 103.0)
- moved C1 56.9 mm to (206.4, 109.5)
- moved R1 56.9 mm to (206.4, 105.5)
- moved R2 56.9 mm to (206.4, 107.5)
- moved R3 56.9 mm to (206.4, 113.6)
- moved R4 56.9 mm to (206.4, 111.6)
- moved U1 56.9 mm to (212.6, 109.5)
- moved R5 55.7 mm to (221.3, 106.6), turned to 0 degrees
- moved C2 55.7 mm to (217.8, 110.8), turned to -90 degrees
- moved F3 55.6 mm to (222.1, 110.3)
- moved J2 54.0 mm to (227.5, 104.1)
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Connections:
- net Net-(U3-XTAL1/PB6) renamed /Clock+
- net Net-(U3-XTAL2/PB7) renamed /Clock-
Routing:
- net GND: track 23.5 -> 46.9 mm
- net LEAD_1: track 25.0 -> 4.45 mm
- net LEAD_2: track 24.6 -> 4.65 mm
- net Net-(U3-~{RESET}/PC6): track 4.27 -> 18.6 mm
- net Net-(F2-Pad2): track 3.06 -> 16.5 mm
- net Net-(F1-Pad2): track 3.31 -> 16.3 mm
- net /Clock-: track 0.00 -> 9.64 mm
- net /Clock+: track 0.00 -> 9.62 mm
- net Net-(D4-K): track 0.00 -> 2.80 mm
- net LEAD_3: track 6.32 -> 4.38 mm
- net LEAD_4: track 17.3 -> 16.2 mm, vias 0 -> 1
Other:
- board text added: "FUSE(500mA) SHUNT(0.01Ω) FUSE(1A) FUSE(500mA)"
- board text added: "Open Source Hardware Enterprise Mini-DMM"
- board text removed: "FUSE(1A)"
- board text removed: "FUSE(500mA)"
- board text removed: "Open Source Hardware Enterprise Mini-DMM OSHE.IO"

Commit message: Finished PCB
Parts:
- removed the G*** at (200.0, 149.0)
- removed the J3 at (104.5, 80.0)
- removed the R10 at (159.3, 83.5)
- removed the R11 at (161.3, 83.5)
- added J1: FTDI Basic, Connector_PinHeader_2.54mm:PinHeader_1x06_P2.54mm_Horizontal, F.Cu at (168.3, 81.1)
- added J4: TEST LEAD CONNECTIONS, Connector_PinHeader_2.54mm:PinHeader_1x04_P2.54mm_Horizontal, F.Cu at (168.3, 121.2)
- C10: renamed from C7; value 1uF -> 10uF
- C8: renamed from C4; value 1uF -> 10uF
- C9: renamed from C6; value 1uF -> 10uF
- J2: value TEST LEAD CONNECTIONS -> ICSP; footprint Connector_PinHeader_2.54mm:PinHeader_1x06_P2.54mm_Horizontal -> Connector_PinHeader_2.54mm:PinHeader_2x03_P2.54mm_Horizontal
- SW1: value MODE SELECT -> PTS526 SK15 SMTR2 LFS
- moved J2 89.2 mm to (138.7, 96.2), turned to 180 degrees
- moved C6 61.6 mm to (147.2, 126.6)
- moved C7 61.6 mm to (158.7, 127.9)
- moved R1 61.6 mm to (147.2, 122.5)
- moved R2 61.6 mm to (147.2, 124.6)
- moved R3 61.6 mm to (147.2, 130.7)
- moved R4 61.6 mm to (147.2, 128.6)
- moved R5 61.6 mm to (162.2, 123.7)
- moved F1 61.6 mm to (162.9, 120.0)
- moved F2 61.6 mm to (162.9, 130.6)
- moved F3 61.6 mm to (162.9, 127.4)
- moved U1 61.6 mm to (153.5, 126.6)
- moved C3 61.1 mm to (165.2, 82.1), turned to 90 degrees
- moved R11 60.7 mm to (165.2, 87.7), turned to -90 degrees
- moved C5 60.1 mm to (139.1, 137.8), turned to 90 degrees
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- renumbered C3 to C1, C5 to C2, C8 to C3, C9 to C4, C10 to C5, C1 to C6, C2 to C7, J1 to J3, R12 to R10, R13 to R11, U3 to U2, U2 to U3
Connections:
- C3 pad 1: Net-(U3-~{RESET}/PC6) -> RESET
- D1 pad 2: D2 -> D7
- D2 pad 2: D3 -> D6
- D3 pad 2: D4 -> D5
- D4 pad 2: D5 -> D9
- J2 pad 1: LEAD_1 -> MISO/D12
- J2 pad 2: LEAD_4 -> MOSI/D11
- J2 pad 3: LEAD_3 -> SCK/D13
- J2 pad 4: LEAD_2 -> RESET
- J2 pad 5: unconnected-(J2-Pin_5-Pad5) -> +3.3V
- J2 pad 6: unconnected-(J2-Pin_6-Pad6) -> GND
- R11 pad 1: Net-(U3-~{RESET}/PC6) -> RESET
- SW1 pad 1: D6 -> D8
- SW1 pad 2: GND -> D8
- SW1 pad 3: (no net) -> GND
- SW1 pad 4: (no net) -> GND
- SW2 pad 1: Net-(U3-~{RESET}/PC6) -> RESET
- SW2 pad 2: Net-(U3-~{RESET}/PC6) -> RESET
- U1 pad 13: A3 -> A2
- U1 pad 14: A3 -> A2
- U1 pad 8: A2 -> A3
- U1 pad 9: A2 -> A3
- U2 pad 29: Net-(U3-~{RESET}/PC6) -> RESET
- U3 pad 23: Net-(U2-VLCD) -> GND
Routing:
- net RESET: track 0.00 -> 117.8 mm, vias 0 -> 2
- net TXD: track 0.00 -> 111.9 mm, vias 0 -> 1
- net RXD: track 0.00 -> 105.5 mm, vias 0 -> 1
- net A5/SCL: track 0.00 -> 78.2 mm
- net A4/SDA: track 0.00 -> 74.4 mm
- net D7: track 0.00 -> 68.3 mm
- net D6: track 0.00 -> 65.7 mm
- net D5: track 0.00 -> 63.2 mm
- net D9: track 0.00 -> 55.6 mm
- net GND: track 46.9 -> 89.7 mm, vias 0 -> 15
- net D8: track 0.00 -> 40.1 mm
- net A2: track 1.27 -> 39.8 mm, vias 0 -> 2
- net A3: track 1.27 -> 34.9 mm, vias 0 -> 2
- net MOSI/D11: track 0.00 -> 33.1 mm
- net A1: track 1.27 -> 28.3 mm, vias 0 -> 2
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- added copper zone on B.Cu, net GND
Other:
- board text added: "ISCP"
- board text added: "MODE"
- board text added: "MODE SELECT"
- board text added: "Open Source Hardware Enterprise Mini Digital Multimeter"
- board text added: "PROGRAMMING"
- board text added: "Pins: 1: Voltage + 2: Current + 3: Current - 4: Voltage -"
- board text removed: "Open Source Hardware Enterprise Mini-DMM"

Commit message: Exported final board
Routing:
- net GND: track 89.7 -> 79.1 mm
- added copper zone on F.Cu, net GND
Changed lines of the file:
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@@
 			(size 1 1)
 			(drill 1)
-			(layers "F&B.Cu" "*.Mask")
+			(layers "*.Cu" "*.Mask")
 		)
 		(pad "" np_thru_hole circle
@@
 			(size 1 1)
 			(drill 1)
-			(layers "F&B.Cu" "*.Mask")
+			(layers "*.Cu" "*.Mask")
 		)
 		(pad "1" smd rect
@@
 	)
 	(segment
-		(start 150.3758 76.727)
-		(end 150.3754 76.7266)
-		(width 0.381)
-		(layer "F.Cu")
-		(net 2)
-	)
-	(segment
-		(start 151.1758 76.739)
-		(end 151.1882 76.7266)
-		(width 0.381)
-		(layer "F.Cu")
-		(net 2)
-	)
-	(segment
 		(start 146.1421 126.5936)
 		(end 146.1513 126.6028)
@@
 	)
 	(segment
-		(start 149.5758 76.7388)
-		(end 149.588 76.7266)
-		(width 0.381)
-		(layer "F.Cu")
-		(net 2)
-	)
-	(segment
 		(start 132.6681 115.4684)
 		(end 132.6681 115.2945)
@@
 	)
 	(segment
-		(start 151.1758 78.0864)
-		(end 151.1758 76.739)
-		(width 0.381)
-		(layer "F.Cu")
-		(net 2)
-	)
-	(segment
 		(start 137.405 113.3602)
 		(end 134.62 113.3602)
@@
 	)
 	(segment
-		(start 153.197 76.7266)
-		(end 151.9756 76.7266)
-		(width 0.381)
-		(layer "F.Cu")
-		(net 2)
-	)
-	(segment
 		(start 174.7468 71.3232)
 		(end 174.736 71.334)
@@
 	)
 	(segment
-		(start 153.5758 77.1054)
-		(end 153.197 76.7266)
-		(width 0.381)
-		(layer "F.Cu")
-		(net 2)
-	)
-	(segment
 		(start 174.7308 67.7672)
 		(end 174.72 67.778)
@@
 	)
 	(segment
-		(start 150.3754 76.7266)
-		(end 149.588 76.7266)
-		(width 0.381)
-		(layer "F.Cu")
-		(net 2)
-	)
-	(segment
 		(start 146.1513 126.6028)
 		(end 146.1513 124.6083)
@@
 	)
 	(segment
-		(start 151.9758 76.7268)
-		(end 151.9756 76.7266)
-		(width 0.381)
-		(layer "F.Cu")
-		(net 2)
-	)
-	(segment
 		(start 156.8704 98.3234)
 		(end 155.702 99.4918)
@@
 	)
 	(segment
-		(start 150.3758 78.0864)
-		(end 150.3758 76.727)
-		(width 0.381)
-		(layer "F.Cu")
-		(net 2)
-	)
-	(segment
 		(start 134.62 113.3602)
 		(end 132.6681 115.3121)
@@
 	)
 	(segment
-		(start 151.1882 76.7266)
-		(end 150.3754 76.7266)
-		(width 0.381)
-		(layer "F.Cu")
-		(net 2)
-	)
-	(segment
 		(start 131.2672 113.8936)
 		(end 131.2672 112.98555)
@@
 	)
 	(segment
-		(start 151.9756 76.7266)
-		(end 151.1882 76.7266)
-		(width 0.381)
-		(layer "F.Cu")
-		(net 2)
-	)
-	(segment
-		(start 151.9758 78.0864)
-		(end 151.9758 76.7268)
-		(width 0.381)
-		(layer "F.Cu")
-		(net 2)
-	)
-	(segment
 		(start 153.1874 89.0524)
 		(end 156.8704 92.7354)
@@
 	)
 	(segment
-		(start 149.5758 78.0864)
-		(end 149.5758 76.7388)
-		(width 0.381)
-		(layer "F.Cu")
-		(net 2)
-	)
-	(segment
 		(start 133.1763 126.63815)
 		(end 133.1662 126.62805)
@@
 	)
 	(segment
-		(start 153.5758 78.0864)
-		(end 153.5758 77.1054)
-		(width 0.381)
-		(layer "F.Cu")
-		(net 2)
-	)
-	(segment
 		(start 155.702 99.4918)
 		(end 155.47975 99.4918)
@@
 	)
 	(via
-		(at 149.588 76.7266)
+		(at 149.6822 76.7588)
 		(size 0.6096)
 		(drill 0.3048)
@@
 	)
 	(zone
+		(net 2)
+		(net_name "GND")
+		(layer "F.Cu")
+		(hatch edge 0.5)
+		(priority 3)
+		(connect_pads yes
+			(clearance 0.254)
+		)
+		(min_thickness 0.25)
+		(filled_areas_thickness no)
+		(fill yes
+			(thermal_gap 0.5)
+			(thermal_bridge_width 0.5)
+		)
+		(polygon
+			(pts
+				(xy 149.3012 78.6892) (xy 152.2222 78.6892) (xy 152.2222 77.216) (xy 153.3144 77.216) (xy 153.3144 78.6892)
+				(xy 153.8224 78.6892) (xy 153.8224 76.3778) (xy 149.3012 76.3778)
+			)
+		)
+	)
+	(zone
