File: mini_dmm/mini_dmm_KiCAD/oshe_mini_dmm_project/oshe_mini_dmm_project.kicad_sch (KiCad schematic)
At the start: 42 parts, among them J1 FTDI Basic, J2 ICSP, J3 DISPLAY, J4 TEST LEAD CONNECTIONS, SW1 PTS526 SK15 SMTR2 LFS, SW2 PTS526 SK15 SMTR2 LFS, SW3 SW_DPDT_x2, U1 LM324, U2 ATmega328P-A, U3 BU91796FS-ME2, U4 LM2664M6, Y1 16MHz

Commit message: Updated files to latest
Parts:
- added C11: 0.1uF, Capacitor_SMD:C_0805_2012Metric_Pad1.18x1.45mm_HandSolder, symbol Device:C
- added R12, R15: 100k, Resistor_SMD:R_0805_2012Metric_Pad1.20x1.40mm_HandSolder, symbol Device:R_US
- added R13, R14, R16: 10k, Resistor_SMD:R_0805_2012Metric_Pad1.20x1.40mm_HandSolder, symbol Device:R_US
Connections:
- net A2: no longer U1.13 (-), U1.14
- net A3: now also C11.2, R12.1; no longer U1.9 (-)
- net GND: now also C11.1, R15.2, R16.2
- net LEAD_4: now also R13.2; no longer U1.12 (+)
- net at F3.2, R5.1: now also R14.2; no longer U1.10 (+)
- new net: R14.1, R15.1, U1.10 (+)
- new net: R12.2, R13.1, U1.9 (-)
- new net: R16.1, U1.12 (+)
- new net: U1.13 (-), U1.14
Other:
- note added: "NOTE: Battery draw appears to be excessive, op-amps clamping on original board?"
- moved on the sheet: F3, R5, U1C, U1D
